Commit message: 4wheel ver

File: urdf/my_robot.urdf (robot description, URDF)
Before this commit: robot four_wheeled_robot, 7 links, 6 joints
Links:
- link base_link: geometry collision box size=0.4 0.5 0.1; visual box size=0.4 0.5 0.1
- link body_top: geometry collision box size=0.4 0.5 0.2; visual box size=0.4 0.5 0.2
Joints:
- joint joint_wheel_bl: origin xyz=-0.15 0.15 -0.05 rpy=0 1.570796326795 0 -> xyz=-0.2 -0.174 -0.05 rpy=0 -1.570796326795 0
- joint joint_wheel_br: origin xyz=-0.15 -0.15 -0.05 rpy=0 1.570796326795 0 -> xyz=0.2 -0.174 -0.05 rpy=0 -1.570796326795 0
- joint joint_wheel_fl: origin xyz=0.15 0.15 -0.05 rpy=0 1.570796326795 0 -> xyz=-0.2 0.174 -0.05 rpy=0 -1.570796326795 0
- joint joint_wheel_fr: origin xyz=0.15 -0.15 -0.05 rpy=0 1.570796326795 0 -> xyz=0.2 0.174 -0.05 rpy=0 -1.570796326795 0

File: urdf/my_robot.xacro (robot description, xacro)
@@ -2,6 +2,6 @@
     <xacro:property name="PI" value="3.14159265359" />
     <!-- Parameters -->
-    <xacro:property name="chassis_length" value="0.3" /> <!-- 30 cm -->
-    <xacro:property name="chassis_width" value="0.3" />  <!-- 30 cm -->
+    <xacro:property name="chassis_length" value="0.5" /> <!-- 50 cm -->
+    <xacro:property name="chassis_width" value="0.4" />  <!-- 40 cm -->
     <xacro:property name="chassis_height" value="0.1" /> <!-- 10 cm -->
     <xacro:property name="wheel_diameter" value="0.152" /> <!-- 15.2 cm -->
@@ -11,6 +11,6 @@
     <xacro:property name="telescopic_rod_max_length" value="0.3" /> <!-- 30 cm -->
     <xacro:property name="telescopic_rod_radius" value="0.02" /> <!-- 2 cm -->
-    <xacro:property name="body_top_length" value="0.3" /> <!-- 30 cm -->
-    <xacro:property name="body_top_width" value="0.3" />  <!-- 30 cm -->
+    <xacro:property name="body_top_length" value="0.5" /> <!-- 30 cm -->
+    <xacro:property name="body_top_width" value="0.4" />  <!-- 30 cm -->
     <xacro:property name="body_top_height" value="0.2" /> <!-- 20 cm -->
     <!-- Base Link -->
@@ -18,5 +18,5 @@
         <visual>
             <geometry>
-                <box size="${chassis_length} ${chassis_width} ${chassis_height}" />
+                <box size="${chassis_width} ${chassis_length} ${chassis_height}" />
             </geometry>
             <material name="gray" />
@@ -24,5 +24,5 @@
         <collision>
             <geometry>
-                <box size="${chassis_length} ${chassis_width} ${chassis_height}" />
+                <box size="${chassis_width} ${chassis_length} ${chassis_height}" />
             </geometry>
         </collision>
@@ -110,5 +110,6 @@
         <parent link="base_link" />
         <child link="wheel_fl" />
-        <origin xyz="${chassis_length/2} ${chassis_width/2} -${chassis_height/2}" rpy="0 ${PI/2} 0" /> <!--
+        <origin xyz="${-chassis_width/2} ${chassis_length/2-wheel_radius} -${chassis_height/2}"
+            rpy="0 ${-PI/2} 0" /> <!--
         Place wheel at the front-left corner -->
         <axis xyz="0 0 1" />
@@ -117,5 +118,6 @@
         <parent link="base_link" />
         <child link="wheel_fr" />
-        <origin xyz="${chassis_length/2} -${chassis_width/2} -${chassis_height/2}" rpy="0 ${PI/2} 0" /> <!--
+        <origin xyz="${chassis_width/2} ${chassis_length/2-wheel_radius} -${chassis_height/2}"
+            rpy="0 ${-PI/2} 0" /> <!--
         Place wheel at the front-right corner -->
         <axis xyz="0 0 1" />
@@ -124,5 +126,6 @@
         <parent link="base_link" />
         <child link="wheel_bl" />
-        <origin xyz="-${chassis_length/2} ${chassis_width/2} -${chassis_height/2}" rpy="0 ${PI/2} 0" /> <!--
+        <origin xyz="${-chassis_width/2} -${chassis_length/2-wheel_radius} -${chassis_height/2}"
+            rpy="0 ${-PI/2} 0" /> <!--
         Place wheel at the back-left corner -->
         <axis xyz="0 0 1" />
@@ -131,6 +134,6 @@
         <parent link="base_link" />
         <child link="wheel_br" />
-        <origin xyz="-${chassis_length/2} -${chassis_width/2} -${chassis_height/2}"
-            rpy="0 ${PI/2} 0" /> <!-- Place wheel at the back-right corner -->
+        <origin xyz="${chassis_width/2} -${chassis_length/2-wheel_radius} -${chassis_height/2}"
+            rpy="0 ${-PI/2} 0" /> <!-- Place wheel at the back-right corner -->
         <axis xyz="0 0 1" />
     </joint>
@@ -164,5 +167,5 @@
         <visual>
             <geometry>
-                <box size="${body_top_length} ${body_top_width} ${body_top_height}" />
+                <box size="${body_top_width} ${body_top_length} ${body_top_height}" />
             </geometry>
             <material name="blue" />
@@ -170,5 +173,5 @@
         <collision>
             <geometry>
-                <box size="${body_top_length} ${body_top_width} ${body_top_height}" />
+                <box size="${body_top_width} ${body_top_length} ${body_top_height}" />
             </geometry>
         </collision>
@@ -239,7 +242,7 @@
             <rightJoint>joint_wheel_br</rightJoint>
             <rightJoint>joint_wheel_fr</rightJoint>
-            <wheelSeparation>0.3</wheelSeparation>
-            <wheelDiameter>0.152</wheelDiameter>
-            <torque>5.0</torque>
+            <wheelSeparation>${chassis_width}</wheelSeparation>
+            <wheelDiameter>${wheel_diameter}</wheelDiameter>
+            <torque>0.5</torque>
         </plugin>
     </gazebo>

Commit message: keyboard control

File: urdf/my_robot.urdf (robot description, URDF)
Before this commit: robot four_wheeled_robot, 7 links, 6 joints
Links:
- removed link wheel_bl
- removed link wheel_br
- removed link wheel_fl
- removed link wheel_fr
- added link base_footprint; visual sphere radius=0.001
- added link body_top_semantic; collision sphere radius=0.05; visual sphere radius=0.05
- added link caster_backward; collision sphere radius=0.03; visual sphere radius=0.03
- added link caster_forward; collision sphere radius=0.03; visual sphere radius=0.03
- added link wheel_left, mass 1.0; collision cylinder length=0.02 radius=0.076; visual cylinder length=0.02 radius=0.076
- added link wheel_right, mass 1.0; collision cylinder length=0.02 radius=0.076; visual cylinder length=0.02 radius=0.076
- link base_link: geometry collision box size=0.4 0.1 0.01; visual box size=0.4 0.1 0.01
- link body_top: geometry collision box size=0.4 0.4 0.2; visual box size=0.4 0.4 0.2
- link telescopic_rod: geometry collision cylinder length=0.3 radius=0.03; visual cylinder length=0.3 radius=0.03
Joints:
- removed joint joint_wheel_bl
- removed joint joint_wheel_br
- removed joint joint_wheel_fl
- removed joint joint_wheel_fr
- added joint base_link_footprint: type fixed, parent base_footprint, child base_link, origin xyz=0 0 0.081
- added joint caster_backward_joint: type fixed, parent base_link, child caster_backward, origin xyz=0 -0.020000000000000004 -0.05 rpy=0 0 0
- added joint caster_forward_joint: type fixed, parent base_link, child caster_forward, origin xyz=0 0.020000000000000004 -0.05 rpy=0 0 0
- added joint joint_body_top_semantic: type fixed, parent body_top, child body_top_semantic, origin xyz=0 0.15000000000000002 0.1
- added joint joint_wheel_left: type continuous, parent base_link, child wheel_left, origin xyz=-0.2 0 -0.005 rpy=0 -1.570796326795 0, axis 0 0 1
- added joint joint_wheel_right: type continuous, parent base_link, child wheel_right, origin xyz=0.2 0 -0.005 rpy=0 -1.570796326795 0, axis 0 0 1
- joint joint_telescopic_rod: origin xyz=0 0 0.2 -> xyz=0 0 0.155

File: urdf/my_robot.xacro (robot description, xacro)
@@ -2,16 +2,29 @@
     <xacro:property name="PI" value="3.14159265359" />
     <!-- Parameters -->
-    <xacro:property name="chassis_length" value="0.5" /> <!-- 50 cm -->
+    <xacro:property name="chassis_length" value="0.1" /> <!-- 50 cm -->
     <xacro:property name="chassis_width" value="0.4" />  <!-- 40 cm -->
-    <xacro:property name="chassis_height" value="0.1" /> <!-- 10 cm -->
+    <xacro:property name="chassis_height" value="0.01" /> <!-- 10 cm -->
     <xacro:property name="wheel_diameter" value="0.152" /> <!-- 15.2 cm -->
     <xacro:property name="wheel_radius" value="${wheel_diameter / 2}" />
     <xacro:property name="wheel_width" value="0.02" /> <!-- 2 cm -->
+    <xacro:property name="caster_radius" value="0.03" /> <!-- 15.2 cm -->
     <xacro:property name="telescopic_rod_min_length" value="0.1" /> <!-- 10 cm -->
     <xacro:property name="telescopic_rod_max_length" value="0.3" /> <!-- 30 cm -->
-    <xacro:property name="telescopic_rod_radius" value="0.02" /> <!-- 2 cm -->
-    <xacro:property name="body_top_length" value="0.5" /> <!-- 30 cm -->
+    <xacro:property name="telescopic_rod_radius" value="0.03" /> <!-- 2 cm -->
+    <xacro:property name="body_top_length" value="0.4" /> <!-- 30 cm -->
     <xacro:property name="body_top_width" value="0.4" />  <!-- 30 cm -->
     <xacro:property name="body_top_height" value="0.2" /> <!-- 20 cm -->
+    <!-- <link name="base_footprint">
+        <visual>
+            <geometry>
+                <sphere radius="0.001" />
+            </geometry>
+        </visual>
+    </link>
+    <joint name="base_link_footprint" type="fixed">
+        <parent link="base_footprint" />
+        <child link="base_link" />
+        <origin xyz="0 0 ${chassis_height/2+wheel_radius}" />
+    </joint> -->
     <!-- Base Link -->
     <link name="base_link">
@@ -34,5 +47,5 @@
     </link>
     <!-- Four Wheels -->
-    <link name="wheel_fl">
+    <link name="wheel_left">
         <visual>
             <geometry>
@@ -52,5 +65,5 @@
         </inertial>
     </link>
-    <link name="wheel_fr">
+    <link name="wheel_right">
         <visual>
             <geometry>
@@ -70,71 +83,70 @@
         </inertial>
     </link>
-    <link name="wheel_bl">
-        <visual>
-            <geometry>
-                <cylinder radius="${wheel_radius}" length="${wheel_width}" />
-            </geometry>
-            <material name="black" />
-        </visual>
-        <collision>
-            <geometry>
-                <cylinder radius="${wheel_radius}" length="${wheel_width}" />
-            </geometry>
-        </collision>
-        <inertial>
-            <mass value="1.0" />
-            <origin xyz="0 0 0" />
-            <inertia ixx="0.01" ixy="0.0" ixz="0.0" iyy="0.01" iyz="0.0" izz="0.01" />
-        </inertial>
-    </link>
-    <link name="wheel_br">
-        <visual>
-            <geometry>
-                <cylinder radius="${wheel_radius}" length="${wheel_width}" />
-            </geometry>
-            <material name="black" />
-        </visual>
-        <collision>
-            <geometry>
-                <cylinder radius="${wheel_radius}" length="${wheel_width}" />
-            </geometry>
-        </collision>
-        <inertial>
-            <mass value="1.0" />
-            <origin xyz="0 0 0" />
-            <inertia ixx="0.01" ixy="0.0" ixz="0.0" iyy="0.01" iyz="0.0" izz="0.01" />
-        </inertial>
-    </link>
     <!-- Joints for Wheels -->
-    <joint name="joint_wheel_fl" type="continuous">
-        <parent link="base_link" />
-        <child link="wheel_fl" />
-        <origin xyz="${-chassis_width/2} ${chassis_length/2-wheel_radius} -${chassis_height/2}"
-            rpy="0 ${-PI/2} 0" /> <!--
-        Place wheel at the front-left corner -->
+    <joint name="joint_wheel_left" type="continuous">
+        <parent link="base_link" />
+        <child link="wheel_left" />
+        <origin xyz="${-chassis_width/2} 0 -${chassis_height/2}"
+            rpy="0 ${-PI/2} 0" />
         <axis xyz="0 0 1" />
     </joint>
-    <joint name="joint_wheel_fr" type="continuous">
-        <parent link="base_link" />
-        <child link="wheel_fr" />
-        <origin xyz="${chassis_width/2} ${chassis_length/2-wheel_radius} -${chassis_height/2}"
-            rpy="0 ${-PI/2} 0" /> <!--
-        Place wheel at the front-right corner -->
+    <joint name="joint_wheel_right" type="continuous">
+        <parent link="base_link" />
+        <child link="wheel_right" />
+        <origin xyz="${chassis_width/2} 0 -${chassis_height/2}"
+            rpy="0 ${-PI/2} 0" />
         <axis xyz="0 0 1" />
     </joint>
-    <joint name="joint_wheel_bl" type="continuous">
-        <parent link="base_link" />
-        <child link="wheel_bl" />
-        <origin xyz="${-chassis_width/2} -${chassis_length/2-wheel_radius} -${chassis_height/2}"
-            rpy="0 ${-PI/2} 0" /> <!--
-        Place wheel at the back-left corner -->
-        <axis xyz="0 0 1" />
-    </joint>
-    <joint name="joint_wheel_br" type="continuous">
-        <parent link="base_link" />
-        <child link="wheel_br" />
-        <origin xyz="${chassis_width/2} -${chassis_length/2-wheel_radius} -${chassis_height/2}"
-            rpy="0 ${-PI/2} 0" /> <!-- Place wheel at the back-right corner -->
-        <axis xyz="0 0 1" />
+    <link name="caster_forward">
+        <!-- <visual>
+            <geometry>
+                <sphere radius="${caster_radius}" />
+            </geometry>
+            <origin xyz="0 0 0" rpy="0 0 0" />
+            <material name="green" />
+        </visual> -->
+        <collision>
+            <origin rpy="0 0 0" xyz="0 0 0" />
+            <geometry>
+                <sphere radius="${caster_radius}" />
+            </geometry>
+        </collision>
+        <!-- <inertial>
+            <mass value="0.5" />
+            <inertia ixx="3.000e-4" iyy="3.000e-4" izz="3.000e-4" ixy="0" ixz="0" iyz="0" />
+        </inertial> -->
+    </link>
+    <link name="caster_backward">
+        <!-- <visual>
+            <geometry>
+                <sphere radius="${caster_radius}" />
+            </geometry>
+            <origin xyz="0 0 0" rpy="0 0 0" />
+            <material name="green" />
+        </visual> -->
+        <collision>
+            <origin rpy="0 0 0" xyz="0 0 0" />
+            <geometry>
+                <sphere radius="${caster_radius}" />
+            </geometry>
+        </collision>
+        <!-- <inertial>
+            <mass value="0.5" />
+            <inertia ixx="3.000e-4" iyy="3.000e-4" izz="3.000e-4" ixy="0" ixz="0" iyz="0" />
+        </inertial> -->
+    </link>
+    <joint name="caster_forward_joint" type="fixed">
+        <origin
+            xyz="0 ${body_top_length/2-caster_radius} ${-chassis_height/2-wheel_radius+caster_radius}"
+            rpy="0 0 0" />
+        <parent link="base_link" />
+        <child link="caster_forward" />
+    </joint>
+    <joint name="caster_backward_joint" type="fixed">
+        <origin
+            xyz="0 ${-body_top_length/2+caster_radius} ${-chassis_height/2-wheel_radius+caster_radius}"
+            rpy="0 0 0" />
+        <parent link="base_link" />
+        <child link="caster_backward" />
     </joint>
     <!-- Telescopic Rod -->
@@ -193,38 +205,39 @@
             effort="10.0" velocity="0.05" /> <!-- 10 cm to 30 cm -->
     </joint>
+    <link name="body_top_semantic">
+        <visual>
+            <geometry>
+                <sphere radius="${body_top_width/8}" />
+            </geometry>
+            <material name="black" />
+        </visual>
+        <collision>
+            <geometry>
+                <sphere radius="${body_top_width/8}" />
+            </geometry>
+        </collision>
+    </link>
+    <joint name="joint_body_top_semantic" type="fixed">
+        <parent link="body_top" />
+        <child link="body_top_semantic" />
+        <origin
+            xyz="0 ${body_top_length/2-body_top_width/8} ${body_top_height/2}" />
+    </joint>
     <!-- Transmission for the wheels -->
-    <transmission name="trans_wheel_fl">
+    <transmission name="trans_wheel_left">
         <type>transmission_interface/SimpleTransmission</type>
-        <joint name="joint_wheel_fl">
+        <joint name="joint_wheel_left">
             <hardwareInterface>hardware_interface/VelocityJointInterface</hardwareInterface>
         </joint>
-        <actuator name="actuator_wheel_fl">
+        <actuator name="actuator_wheel_left">
             <mechanicalReduction>1</mechanicalReduction>
         </actuator>
     </transmission>
-    <transmission name="trans_wheel_fr">
+    <transmission name="trans_wheel_right">
         <type>transmission_interface/SimpleTransmission</type>
-        <joint name="joint_wheel_fr">
+        <joint name="joint_wheel_right">
             <hardwareInterface>hardware_interface/VelocityJointInterface</hardwareInterface>
         </joint>
-        <actuator name="actuator_wheel_fr">
-            <mechanicalReduction>1</mechanicalReduction>
-        </actuator>
-    </transmission>
-    <transmission name="trans_wheel_bl">
-        <type>transmission_interface/SimpleTransmission</type>
-        <joint name="joint_wheel_bl">
-            <hardwareInterface>hardware_interface/VelocityJointInterface</hardwareInterface>
-        </joint>
-        <actuator name="actuator_wheel_bl">
-            <mechanicalReduction>1</mechanicalReduction>
-        </actuator>
-    </transmission>
-    <transmission name="trans_wheel_br">
-        <type>transmission_interface/SimpleTransmission</type>
-        <joint name="joint_wheel_br">
-            <hardwareInterface>hardware_interface/VelocityJointInterface</hardwareInterface>
-        </joint>
-        <actuator name="actuator_wheel_br">
+        <actuator name="actuator_wheel_right">
             <mechanicalReduction>1</mechanicalReduction>
         </actuator>
@@ -238,12 +251,36 @@
             </ros>
             <updateRate>50</updateRate>
-            <leftJoint>joint_wheel_bl</leftJoint>
-            <leftJoint>joint_wheel_fl</leftJoint>
-            <rightJoint>joint_wheel_br</rightJoint>
-            <rightJoint>joint_wheel_fr</rightJoint>
+            <leftJoint>joint_wheel_left</leftJoint>
+            <rightJoint>joint_wheel_right</rightJoint>
             <wheelSeparation>${chassis_width}</wheelSeparation>
             <wheelDiameter>${wheel_diameter}</wheelDiameter>
-            <torque>0.5</torque>
+            <torque>5</torque>
         </plugin>
     </gazebo>
+    <gazebo reference="base_link">
+        <material>Gazebo/Grey</material>
+    </gazebo>
+    <gazebo reference="wheel_left">
+        <material>Gazebo/DarkGrey</material>
+    </gazebo>
+    <gazebo reference="wheel_right">
+        <material>Gazebo/DarkGrey</material>
+    </gazebo>
+    <gazebo reference="telescopic_rod">
+        <material>Gazebo/White</material>
+    </gazebo>
+    <gazebo reference="body_top">
+        <material>Gazebo/DarkYellow </material>
+    </gazebo>
+    <gazebo reference="body_top_semantic">
+        <material>Gazebo/FlatBlack</material>
+    </gazebo>
+    <gazebo reference="caster_forward">
+        <mu1 value="0.0" />
+        <mu2 value="0.0" />
+    </gazebo>
+    <gazebo reference="caster_backward">
+        <mu1 value="0.0" />
+        <mu2 value="0.0" />
+    </gazebo>
 </robot>
