Commit message: hide base_link

File: urdf/robot.urdf (robot description, URDF)
Before this commit: robot four_wheeled_robot, 9 links, 8 joints
Links:
- removed link base_footprint
- removed link telescopic_rod
- link base_link: mass 10.0 -> None; geometry 
- link caster_backward: geometry collision sphere radius=0.03
- link caster_forward: geometry collision sphere radius=0.03
Joints:
- removed joint base_link_footprint
- removed joint joint_telescopic_rod
- joint caster_backward_joint: origin xyz=0 -0.020000000000000004 -0.05 rpy=0 0 0 -> xyz=0 -0.17 -0.051000000000000004 rpy=0 0 0
- joint caster_forward_joint: origin xyz=0 0.020000000000000004 -0.05 rpy=0 0 0 -> xyz=0 0.17 -0.051000000000000004 rpy=0 0 0
- joint joint_body_top: limit lower=0 upper=0.19999999999999998 effort=10.0 velocity=0.05 -> lower=0.05000000000000002 upper=0.24999999999999997 effort=10.0 velocity=0.05; parent telescopic_rod -> base_link

File: urdf/robot.xacro (robot description, xacro)
@@ -1,43 +1,32 @@
-<robot name="four_wheeled_robot" xmlns:xacro="http://www.ros.org/wiki/xacro">
+<robot name="robot" xmlns:xacro="http://www.ros.org/wiki/xacro">
     <xacro:property name="PI" value="3.14159265359" />
+    <xacro:property name="namespace" value="robot" />
     <!-- Parameters -->
     <xacro:property name="chassis_length" value="0.1" /> <!-- 50 cm -->
     <xacro:property name="chassis_width" value="0.4" />  <!-- 40 cm -->
-    <xacro:property name="chassis_height" value="0.01" /> <!-- 10 cm -->
+    <xacro:property name="chassis_height" value="0.01" /> <!-- 1 cm -->
     <xacro:property name="wheel_diameter" value="0.152" /> <!-- 15.2 cm -->
     <xacro:property name="wheel_radius" value="${wheel_diameter / 2}" />
     <xacro:property name="wheel_width" value="0.02" /> <!-- 2 cm -->
     <xacro:property name="caster_radius" value="0.03" /> <!-- 15.2 cm -->
-    <xacro:property name="telescopic_rod_min_length" value="0.1" /> <!-- 10 cm -->
-    <xacro:property name="telescopic_rod_max_length" value="0.3" /> <!-- 30 cm -->
-    <xacro:property name="telescopic_rod_radius" value="0.03" /> <!-- 2 cm -->
+    <xacro:property name="min_lift_height" value="0.1" /> <!-- 10 cm -->
+    <xacro:property name="max_lift_height" value="0.3" /> <!-- 30 cm -->
+    <!-- <xacro:property name="telescopic_rod_radius" value="0.03" /> -->
     <xacro:property name="body_top_length" value="0.4" /> <!-- 30 cm -->
     <xacro:property name="body_top_width" value="0.4" />  <!-- 30 cm -->
     <xacro:property name="body_top_height" value="0.2" /> <!-- 20 cm -->
-    <!-- <link name="base_footprint">
-        <visual>
-            <geometry>
-                <sphere radius="0.001" />
-            </geometry>
-        </visual>
-    </link>
-    <joint name="base_link_footprint" type="fixed">
-        <parent link="base_footprint" />
-        <child link="base_link" />
-        <origin xyz="0 0 ${chassis_height/2+wheel_radius}" />
-    </joint> -->
     <!-- Base Link -->
     <link name="base_link">
-        <visual>
+        <!-- <visual>
             <geometry>
                 <box size="${chassis_width} ${chassis_length} ${chassis_height}" />
             </geometry>
             <material name="gray" />
-        </visual>
-        <collision>
+        </visual> -->
+        <!-- <collision>
             <geometry>
                 <box size="${chassis_width} ${chassis_length} ${chassis_height}" />
             </geometry>
-        </collision>
+        </collision> -->
         <inertial>
             <mass value="10.0" />
@@ -151,8 +140,8 @@
     </joint>
     <!-- Telescopic Rod -->
-    <link name="telescopic_rod">
-        <visual>
-            <geometry>
-                <cylinder radius="${telescopic_rod_radius}" length="${telescopic_rod_max_length}" />
+    <!-- <link name="telescopic_rod">
+        <visual>
+            <geometry>
+                <cylinder radius="${telescopic_rod_radius}" length="${max_lift_height}" />
             </geometry>
             <material name="silver" />
@@ -160,5 +149,5 @@
         <collision>
             <geometry>
-                <cylinder radius="${telescopic_rod_radius}" length="${telescopic_rod_max_length}" />
+                <cylinder radius="${telescopic_rod_radius}" length="${max_lift_height}" />
             </geometry>
         </collision>
@@ -168,11 +157,11 @@
             <inertia ixx="0.001" ixy="0.0" ixz="0.0" iyy="0.001" iyz="0.0" izz="0.001" />
         </inertial>
-    </link>
+    </link> -->
     <!-- Joint for Telescopic Rod -->
-    <joint name="joint_telescopic_rod" type="fixed">
+    <!-- <joint name="joint_telescopic_rod" type="fixed">
         <parent link="base_link" />
         <child link="telescopic_rod" />
-        <origin xyz="0 0 ${(chassis_height+telescopic_rod_max_length)/2}" /> <!-- Attach rod to the top of the base -->
-    </joint>
+        <origin xyz="0 0 ${(chassis_height+max_lift_height)/2}" />
+    </joint> -->
     <!-- Body Link on Top of Telescopic Rod -->
     <link name="body_top">
@@ -195,12 +184,13 @@
     </link>
     <!-- Joint for Body Top -->
+    <xacro:property name="lift_origin"
+        value="${body_top_height / 2}" />
     <joint name="joint_body_top" type="prismatic">
-        <parent link="telescopic_rod" />
+        <parent link="base_link" />
         <child link="body_top" />
         <origin
-            xyz="0 0 ${(telescopic_rod_max_length + body_top_height) / 2-(telescopic_rod_max_length-telescopic_rod_min_length)}" /> <!-- Attach body to
-        the top of the rod -->
+            xyz="0 0 ${lift_origin}" />
         <axis xyz="0 0 1" />
-        <limit lower="0" upper="${telescopic_rod_max_length-telescopic_rod_min_length}"
+        <limit lower="${min_lift_height}" upper="${max_lift_height}"
             effort="10.0" velocity="0.05" /> <!-- 10 cm to 30 cm -->
     </joint>
@@ -228,5 +218,5 @@
         <type>transmission_interface/SimpleTransmission</type>
         <joint name="joint_wheel_left">
-            <hardwareInterface>hardware_interface/VelocityJointInterface</hardwareInterface>
+            <hardwareInterface>VelocityJointInterface</hardwareInterface>
         </joint>
         <actuator name="actuator_wheel_left">
@@ -237,7 +227,16 @@
         <type>transmission_interface/SimpleTransmission</type>
         <joint name="joint_wheel_right">
-            <hardwareInterface>hardware_interface/VelocityJointInterface</hardwareInterface>
+            <hardwareInterface>VelocityJointInterface</hardwareInterface>
         </joint>
         <actuator name="actuator_wheel_right">
+            <mechanicalReduction>1</mechanicalReduction>
+        </actuator>
+    </transmission>
+    <transmission name="trans_body_top">
+        <type>transmission_interface/SimpleTransmission</type>
+        <joint name="joint_body_top">
+            <hardwareInterface>PositionJointInterface</hardwareInterface>
+        </joint>
+        <actuator name="actuator_body_top">
             <mechanicalReduction>1</mechanicalReduction>
         </actuator>
@@ -247,5 +246,5 @@
         <plugin name="gazebo_ros_diff_drive" filename="libgazebo_ros_diff_drive.so">
             <ros>
-                <namespace>/my_robot</namespace>
+                <namespace>/${namespace}</namespace>
                 <remapping>cmd_vel:=cmd_vel</remapping>
             </ros>

Commit message: xacro ns def

File: urdf/robot.urdf (robot description, URDF)
Before this commit: robot robot, 7 links, 6 joints
Links:
- link base_link: mass None -> 10.0
- link body_top: mass 2.0 -> 0.1
Joints:
- joint joint_body_top: limit lower=0.05000000000000002 upper=0.24999999999999997 effort=10.0 velocity=0.05 -> lower=0.1 upper=0.3 effort=1.0 velocity=0.1; origin xyz=0 0 0.05000000000000002 -> xyz=0 0 0.1

File: urdf/robot.xacro (robot description, xacro)
@@ -1,5 +1,5 @@
 <robot name="robot" xmlns:xacro="http://www.ros.org/wiki/xacro">
     <xacro:property name="PI" value="3.14159265359" />
-    <xacro:property name="namespace" value="robot" />
+    <xacro:arg name="ns" default="robot" />
     <!-- Parameters -->
     <xacro:property name="chassis_length" value="0.1" /> <!-- 50 cm -->
@@ -245,5 +245,5 @@
     <!-- <gazebo>
         <plugin name="gazebo_ros_diff_drive" filename="libgazebo_ros_diff_drive.so">
-            <robotNamespace>/${namespace}</robotNamespace>
+            <robotNamespace>/$(arg ns)</robotNamespace>
             <robotBaseFrame>base_link</robotBaseFrame>
             <updateRate>50</updateRate>
@@ -257,5 +257,5 @@
     <gazebo>
         <plugin name="gazebo_ros_control" filename="libgazebo_ros_control.so">
-            <robotNamespace>/${namespace}</robotNamespace>
+            <robotNamespace>/$(arg ns)</robotNamespace>
         </plugin>
     </gazebo>
@@ -305,5 +305,5 @@
             </ray>
             <plugin name="gazebo_ros_head_ydlidar_controller" filename="libgazebo_ros_gpu_laser.so">
-                <robotNamespace>/${namespace}</robotNamespace>
+                <robotNamespace>/$(arg ns)</robotNamespace>
                 <topicName>scan</topicName>
                 <frameName>body_top_semantic</frameName>
