Commit message: adjust mass

File: urdf/robot.xacro (robot description, xacro)
@@ -178,5 +178,5 @@
         </collision>
         <inertial>
-            <mass value="2.0" />
+            <mass value="0.1" />
             <origin xyz="0 0 0" />
             <inertia ixx="0.02" ixy="0.0" ixz="0.0" iyy="0.02" iyz="0.0" izz="0.02" />

Commit message: model mesh

File: urdf/robot.xacro (robot description, xacro)
@@ -3,17 +3,16 @@
     <xacro:arg name="ns" default="robot" />
     <!-- Parameters -->
-    <xacro:property name="chassis_length" value="0.1" /> <!-- 50 cm -->
-    <xacro:property name="chassis_width" value="0.4" />  <!-- 40 cm -->
-    <xacro:property name="chassis_height" value="0.01" /> <!-- 1 cm -->
-    <xacro:property name="wheel_diameter" value="0.152" /> <!-- 15.2 cm -->
+    <xacro:property name="chassis_length" value="0.1" />
+    <xacro:property name="chassis_width" value="0.4" />
+    <xacro:property name="chassis_height" value="0.01" />
+    <xacro:property name="wheel_diameter" value="0.152" />
     <xacro:property name="wheel_radius" value="${wheel_diameter / 2}" />
-    <xacro:property name="wheel_width" value="0.02" /> <!-- 2 cm -->
-    <xacro:property name="caster_radius" value="0.03" /> <!-- 15.2 cm -->
-    <xacro:property name="min_lift_height" value="0.1" /> <!-- 10 cm -->
-    <xacro:property name="max_lift_height" value="0.3" /> <!-- 30 cm -->
-    <!-- <xacro:property name="telescopic_rod_radius" value="0.03" /> -->
-    <xacro:property name="body_top_length" value="0.4" /> <!-- 30 cm -->
-    <xacro:property name="body_top_width" value="0.4" />  <!-- 30 cm -->
-    <xacro:property name="body_top_height" value="0.2" /> <!-- 20 cm -->
+    <xacro:property name="wheel_width" value="0.046" />
+    <xacro:property name="caster_radius" value="0.03" />
+    <xacro:property name="min_lift_height" value="0.012" />
+    <xacro:property name="max_lift_height" value="0.305" />
+    <xacro:property name="body_top_length" value="0.440" />
+    <xacro:property name="body_top_width" value="0.309" />
+    <xacro:property name="body_top_height" value="0.140" />
     <!-- Base Link -->
     <link name="base_link">
@@ -32,5 +31,5 @@
             <mass value="10.0" />
             <origin xyz="0 0 0" />
-            <inertia ixx="0.1" ixy="0.0" ixz="0.0" iyy="0.1" iyz="0.0" izz="0.1" />
+            <inertia ixx="1" ixy="0.0" ixz="0.0" iyy="1" iyz="0.0" izz="1" />
         </inertial>
     </link>
@@ -139,29 +138,4 @@
         <child link="caster_backward" />
     </joint>
-    <!-- Telescopic Rod -->
-    <!-- <link name="telescopic_rod">
-        <visual>
-            <geometry>
-                <cylinder radius="${telescopic_rod_radius}" length="${max_lift_height}" />
-            </geometry>
-            <material name="silver" />
-        </visual>
-        <collision>
-            <geometry>
-                <cylinder radius="${telescopic_rod_radius}" length="${max_lift_height}" />
-            </geometry>
-        </collision>
-        <inertial>
-            <mass value="0.5" />
-            <origin xyz="0 0 0" />
-            <inertia ixx="0.001" ixy="0.0" ixz="0.0" iyy="0.001" iyz="0.0" izz="0.001" />
-        </inertial>
-    </link> -->
-    <!-- Joint for Telescopic Rod -->
-    <!-- <joint name="joint_telescopic_rod" type="fixed">
-        <parent link="base_link" />
-        <child link="telescopic_rod" />
-        <origin xyz="0 0 ${(chassis_height+max_lift_height)/2}" />
-    </joint> -->
     <!-- Body Link on Top of Telescopic Rod -->
     <link name="body_top">
@@ -242,17 +216,4 @@
         </actuator>
     </transmission>
-    <!-- Gazebo plugin for drive control -->
-    <!-- <gazebo>
-        <plugin name="gazebo_ros_diff_drive" filename="libgazebo_ros_diff_drive.so">
-            <robotNamespace>/$(arg ns)</robotNamespace>
-            <robotBaseFrame>base_link</robotBaseFrame>
-            <updateRate>50</updateRate>
-            <leftJoint>joint_wheel_left</leftJoint>
-            <rightJoint>joint_wheel_right</rightJoint>
-            <wheelSeparation>${chassis_width}</wheelSeparation>
-            <wheelDiameter>${wheel_diameter}</wheelDiameter>
-            <torque>5</torque>
-        </plugin>
-    </gazebo> -->
     <gazebo>
         <plugin name="gazebo_ros_control" filename="libgazebo_ros_control.so">

Commit message: update model&launch config

File: urdf/robot.xacro (robot description, xacro)
@@ -4,5 +4,5 @@
     <!-- Parameters -->
     <xacro:property name="chassis_length" value="0.1" />
-    <xacro:property name="chassis_width" value="0.4" />
+    <xacro:property name="chassis_width" value="0.45" />
     <xacro:property name="chassis_height" value="0.01" />
     <xacro:property name="wheel_diameter" value="0.152" />
@@ -29,7 +29,7 @@
         </collision> -->
         <inertial>
-            <mass value="10.0" />
-            <origin xyz="0 0 0" />
-            <inertia ixx="1" ixy="0.0" ixz="0.0" iyy="1" iyz="0.0" izz="1" />
+            <mass value="5" />
+            <origin xyz="0 0 0" />
+            <inertia ixx="0.01" ixy="0.0" ixz="0.0" iyy="0.01" iyz="0.0" izz="0.001" />
         </inertial>
     </link>
@@ -48,5 +48,5 @@
         </collision>
         <inertial>
-            <mass value="1.0" />
+            <mass value="0.01" />
             <origin xyz="0 0 0" />
             <inertia ixx="0.01" ixy="0.0" ixz="0.0" iyy="0.01" iyz="0.0" izz="0.01" />
@@ -66,5 +66,5 @@
         </collision>
         <inertial>
-            <mass value="1.0" />
+            <mass value="0.01" />
             <origin xyz="0 0 0" />
             <inertia ixx="0.01" ixy="0.0" ixz="0.0" iyy="0.01" iyz="0.0" izz="0.01" />
@@ -72,5 +72,5 @@
     </link>
     <!-- Joints for Wheels -->
-    <joint name="joint_wheel_left" type="continuous">
+    <joint name="joint_wheel_l" type="continuous">
         <parent link="base_link" />
         <child link="wheel_left" />
@@ -79,5 +79,5 @@
         <axis xyz="0 0 1" />
     </joint>
-    <joint name="joint_wheel_right" type="continuous">
+    <joint name="joint_wheel_r" type="continuous">
         <parent link="base_link" />
         <child link="wheel_right" />
@@ -154,5 +154,5 @@
             <mass value="0.1" />
             <origin xyz="0 0 0" />
-            <inertia ixx="0.02" ixy="0.0" ixz="0.0" iyy="0.02" iyz="0.0" izz="0.02" />
+            <inertia ixx="0.002" ixy="0.0" ixz="0.0" iyy="0.002" iyz="0.0" izz="0.002" />
         </inertial>
     </link>
@@ -191,5 +191,5 @@
     <transmission name="trans_wheel_left">
         <type>transmission_interface/SimpleTransmission</type>
-        <joint name="joint_wheel_left">
+        <joint name="joint_wheel_l">
             <hardwareInterface>hardware_interface/VelocityJointInterface</hardwareInterface>
         </joint>
@@ -200,5 +200,5 @@
     <transmission name="trans_wheel_right">
         <type>transmission_interface/SimpleTransmission</type>
-        <joint name="joint_wheel_right">
+        <joint name="joint_wheel_r">
             <hardwareInterface>hardware_interface/VelocityJointInterface</hardwareInterface>
         </joint>
@@ -236,5 +236,5 @@
         <material>Gazebo/DarkYellow </material>
     </gazebo>
-    <gazebo reference="body_top_semantic">
+    <!-- <gazebo reference="body_top_semantic">
         <sensor type="gpu_ray" name="head_ydlidar_sensor">
             <pose>0 0 0 0 0 0</pose>
@@ -257,8 +257,4 @@
                 <noise>
                     <type>gaussian</type>
-                    <!-- Noise parameters based on published spec for Hokuyo laser
-               achieving "+-30mm" accuracy at range < 10m.  A mean of 0.0m and
-               stddev of 0.01m will put 99.7% of samples within 0.03m of the true
-               reading. -->
                     <mean>0.0</mean>
                     <stddev>0.01</stddev>
@@ -272,5 +268,5 @@
         </sensor>
         <material>Gazebo/FlatBlack</material>
-    </gazebo>
+    </gazebo> -->
     <gazebo reference="caster_forward">
         <mu1 value="0.0" />

File: urdf/sw.xacro (robot description, xacro)
@@ -24,5 +24,5 @@
   <link
     name="base_link">
-    <inertial>
+    <!-- <inertial>
       <origin
         xyz="-0.0101783300438887 -8.63948981799645E-09 0.0390008530568618"
@@ -37,4 +37,18 @@
         iyz="1.26514888593879E-10"
         izz="0.142687618659048" />
+    </inertial> -->
+    <inertial>
+      <origin
+        xyz="-0.0101783300438887 -8.63948981799645E-09 0.0390008530568618"
+        rpy="0 0 0" />
+      <mass
+        value="0.678677551342344" />
+      <inertia
+        ixx="0.0710000990521389"
+        ixy="3.51370404321391E-09"
+        ixz="0.000957296781231614"
+        iyy="0.0868439733337961"
+        iyz="1.26514888593879E-10"
+        izz="0.000142687618659048" />
     </inertial>
     <visual>
@@ -65,5 +79,5 @@
         rpy="0 0 0" />
       <mass
-        value="0.162466897479642" />
+        value="0.000162466897479642" />
       <inertia
         ixx="3.86909457658897E-05"
@@ -123,5 +137,5 @@
         rpy="0 0 0" />
       <mass
-        value="0.347077595551188" />
+        value="0.000347077595551188" />
       <inertia
         ixx="0.00107716081650825"
@@ -234,5 +248,5 @@
         rpy="0 0 0" />
       <mass
-        value="0.129894864847223" />
+        value="0.000129894864847223" />
       <inertia
         ixx="2.59618087625984E-05"
@@ -292,5 +306,5 @@
         rpy="0 0 0" />
       <mass
-        value="0.24006664343355" />
+        value="0.00024006664343355" />
       <inertia
         ixx="0.000709486550862449"
@@ -347,8 +361,8 @@
     <inertial>
       <origin
-        xyz="0 0.00988036020187399 0"
-        rpy="0 0 0" />
-      <mass
-        value="0.026831378984772" />
+        xyz="0 0.000988036020187399 0"
+        rpy="0 0 0" />
+      <mass
+        value="0.00026831378984772" />
       <inertia
         ixx="4.30409377850185E-06"
@@ -400,8 +414,8 @@
     <inertial>
       <origin
-        xyz="0 0.00988036020187399 0"
-        rpy="0 0 0" />
-      <mass
-        value="0.026831378984772" />
+        xyz="0 0.000988036020187399 0"
+        rpy="0 0 0" />
+      <mass
+        value="0.00026831378984772" />
       <inertia
         ixx="4.30409377850185E-06"
@@ -456,5 +470,5 @@
         rpy="0 0 0" />
       <mass
-        value="0.162466897479642" />
+        value="0.000162466897479642" />
       <inertia
         ixx="3.86909457658898E-05"
@@ -514,5 +528,5 @@
         rpy="0 0 0" />
       <mass
-        value="0.347077595551188" />
+        value="0.000347077595551188" />
       <inertia
         ixx="0.00107716081650825"
@@ -625,5 +639,5 @@
         rpy="0 0 0" />
       <mass
-        value="0.129894864847223" />
+        value="0.000129894864847223" />
       <inertia
         ixx="2.59618087625984E-05"
@@ -683,5 +697,5 @@
         rpy="0 0 0" />
       <mass
-        value="0.240066643433549" />
+        value="0.000240066643433549" />
       <inertia
         ixx="0.000709486550862448"
@@ -741,5 +755,5 @@
         rpy="0 0 0" />
       <mass
-        value="0.026831378984772" />
+        value="0.000026831378984772" />
       <inertia
         ixx="4.30409377850185E-06"
@@ -794,5 +808,5 @@
         rpy="0 0 0" />
       <mass
-        value="0.026831378984772" />
+        value="0.000026831378984772" />
       <inertia
         ixx="4.30409377850185E-06"
@@ -847,5 +861,5 @@
         rpy="0 0 0" />
       <mass
-        value="0.141168695994094" />
+        value="0.000141168695994094" />
       <inertia
         ixx="8.42336911882901E-05"
@@ -905,5 +919,5 @@
         rpy="0 0 0" />
       <mass
-        value="0.239903536199401" />
+        value="0.000239903536199401" />
       <inertia
         ixx="7.70561826554075E-05"
@@ -963,5 +977,5 @@
         rpy="0 0 0" />
       <mass
-        value="0.157217277786466" />
+        value="0.000157217277786466" />
       <inertia
         ixx="1.93415806521528E-05"
@@ -1021,5 +1035,5 @@
         rpy="0 0 0" />
       <mass
-        value="0.141168695994094" />
+        value="0.000141168695994094" />
       <inertia
         ixx="8.42336911882902E-05"
@@ -1079,5 +1093,5 @@
         rpy="0 0 0" />
       <mass
-        value="0.239903536199401" />
+        value="0.000239903536199401" />
       <inertia
         ixx="7.70561826554075E-05"
@@ -1137,5 +1151,5 @@
         rpy="0 0 0" />
       <mass
-        value="0.157217277786466" />
+        value="0.000157217277786466" />
       <inertia
         ixx="1.93415806521528E-05"
@@ -1201,5 +1215,5 @@
     </collision>
     <inertial>
-      <mass value="0.1" />
+      <mass value="0.001" />
       <origin xyz="0 0 0" />
       <inertia ixx="0.0" ixy="0.0" ixz="0.0" iyy="0.0" iyz="0.0" izz="0.0" />
@@ -1259,5 +1273,5 @@
   <joint name="caster_forward_joint" type="fixed">
     <origin
-      xyz="${body_top_length/2-caster_radius} 0 ${-chassis_height/2-wheel_radius+caster_radius}"
+      xyz="${body_top_length/2-caster_radius} 0 ${-chassis_height/2-wheel_radius+caster_radius+0.0001}"
       rpy="0 0 0" />
     <parent link="chassis" />
@@ -1266,5 +1280,5 @@
   <joint name="caster_backward_joint" type="fixed">
     <origin
-      xyz="${-body_top_length/2+caster_radius} 0 ${-chassis_height/2-wheel_radius+caster_radius}"
+      xyz="${-body_top_length/2+caster_radius} 0 ${-chassis_height/2-wheel_radius+caster_radius+0.0001}"
       rpy="0 0 0" />
     <parent link="chassis" />
@@ -1312,3 +1326,20 @@
     <mu2 value="0.0" />
   </gazebo>
+  <gazebo reference="link_wheel_l">
+    <mu1 value="2.0" />
+    <mu2 value="2.0" />
+  </gazebo>
+  <gazebo reference="link_wheel_r">
+    <mu1 value="2.0" />
+    <mu2 value="2.0" />
+  </gazebo>
+  <!-- <xacro:include filename="$(find urdf_simulate)/urdf/livox_mid360.xacro" />
+  <xacro:Livox_Mid360 name="livox" />
+  <joint name="joint_livox" type="fixed">
+    <parent link="base_link" />
+    <child link="livox_base" />
+    <origin
+      xyz="0 0 ${body_top_height}" />
+    <axis xyz="0 0 1" />
+  </joint> -->
 </robot>
